File: phone/phone.kicad_sch (KiCad schematic)
At the start: 4 parts, among them M1 Conn_01x06

Commit message: ADDED SWITCH, LED, CAHRGIN IC AND BATTERY PROTECTION
Parts:
- added B_RAW, LED1, PWR, SW1, SW2, SW3: Conn_01x02, symbol Connector_Generic:Conn_01x02
- added TP4056: Conn_01x04, symbol Connector_Generic:Conn_01x04
- added TPS61023: Conn_01x03, symbol Connector_Generic:Conn_01x03
Connections:
- net 3V3: now also A1.7 (Pin_7)
- net GND: now also B_RAW.2 (Pin_2), SW1.1 (Pin_1), SW2.1 (Pin_1), SW3.1 (Pin_1), TP4056.1 (Pin_1), TP4056.2 (Pin_2), TPS61023.2 (Pin_2)
- net VIN: now also PWR.1 (Pin_1), PWR.2 (Pin_2), TPS61023.3 (Pin_3); no longer A1.7 (Pin_7)
- new net BAT_BOOST: TP4056.4 (Pin_4), TPS61023.1 (Pin_1)
- new net BAT_RAW: B_RAW.1 (Pin_1), TP4056.3 (Pin_3)
- new net SW1: SW1.2 (Pin_2)
- new net SW2: SW2.2 (Pin_2)
- new net SW3: SW3.2 (Pin_2)

Commit message: ADDED ROATRY ENCODER
Parts:
- removed LED1: Conn_01x02, symbol Connector_Generic:Conn_01x02
- added J1: Conn_01x02, solderwirepad_1_02_SMD:SolderWirePad_1x02_SMD_5x5mm, symbol Connector_Generic:Conn_01x02
- added R1: R, symbol Device:R
- added SW4: RotaryEncoder_Switch, symbol Device:RotaryEncoder_Switch
- A1: footprint (none) -> solderwirepad_1_02_SMD:SolderWirePad_1x07_SMD_1x3mm
- M1: footprint (none) -> solderwirepad_1_02_SMD:SolderWirePad_1x06_SMD_1x3mm
- OLED1: renamed from OLED; footprint (none) -> solderwirepad_1_02_SMD:SolderWirePad_1x07_SMD_1x3mm
- PWR1: renamed from PWR; footprint (none) -> solderwirepad_1_02_SMD:SolderWirePad_1x02_SMD_5x5mm
- gave numbers to parts that had none: 1
- renumbered B_RAW to B_RAW1, TP4056 to TP1, TPS61023 to TPS1
Connections:
- net GND: now also J1.1 (Pin_1), SW4.C, SW4.S2
- net SW1: now also U1.J1_15 (GPIO13)
- net SW2: now also U1.J1_11 (GPIO27)
- net SW3: now also U1.J1_12 (GPIO16)
- net LED: now reaches U1.J1_8 (GPIO33)
- net LED: now also R1.2
- net RE_A: now reaches U1.J2_15 (GPIO2)
- net RE_A: now also SW4.A
- net RE_B: now reaches U1.J2_16 (GPIO15)
- net RE_B: now also SW4.B
- new net: J1.2 (Pin_2), R1.1
- new net SW_RE: SW4.S1

Commit message: COMPLETED SCHEMATICS
Parts:
- B_RAW1, SW1, SW2, SW3: footprint (none) -> solderwirepad_1_02_SMD:SolderWirePad_1x02_SMD_5x5mm
- R1: footprint (none) -> Resistor_THT:R_Axial_DIN0207_L6.3mm_D2.5mm_P7.62mm_Horizontal
- SW4: footprint (none) -> solderwirepad_1_02_SMD:SolderWirePad_1x05_SMD_1x3mm
- TP1: footprint (none) -> solderwirepad_1_02_SMD:SolderWirePad_1x04_SMD_1x3mm
- TPS1: footprint (none) -> solderwirepad_1_02_SMD:SolderWirePad_1x03_SMD_1x3mm
Changed lines of the file:
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@@
     (property "Reference" "R1" (id 0) (at 123.19 99.06 90))
     (property "Value" "R" (id 1) (at 123.19 101.6 90))
-    (property "Footprint" "" (id 2) (at 123.19 107.188 90)
+    (property "Footprint" "Resistor_THT:R_Axial_DIN0207_L6.3mm_D2.5mm_P7.62mm_Horizontal" (id 2) (at 123.19 107.188 90)
       (effects (font (size 1.27 1.27)) hide)
     )
@@
       (effects (font (size 1.27 1.27)) (justify left))
     )
-    (property "Footprint" "" (id 2) (at 185.42 86.36 0)
+    (property "Footprint" "solderwirepad_1_02_SMD:SolderWirePad_1x04_SMD_1x3mm" (id 2) (at 185.42 86.36 0)
       (effects (font (size 1.27 1.27)) hide)
     )
@@
     (property "Reference" "SW2" (id 0) (at 135.89 81.28 0))
     (property "Value" "Conn_01x02" (id 1) (at 135.89 83.82 0))
-    (property "Footprint" "" (id 2) (at 135.89 90.17 0)
+    (property "Footprint" "solderwirepad_1_02_SMD:SolderWirePad_1x02_SMD_5x5mm" (id 2) (at 135.89 90.17 0)
       (effects (font (size 1.27 1.27)) hide)
     )
@@
     (property "Reference" "SW3" (id 0) (at 151.13 81.28 0))
     (property "Value" "Conn_01x02" (id 1) (at 151.13 83.82 0))
-    (property "Footprint" "" (id 2) (at 151.13 90.17 0)
+    (property "Footprint" "solderwirepad_1_02_SMD:SolderWirePad_1x02_SMD_5x5mm" (id 2) (at 151.13 90.17 0)
       (effects (font (size 1.27 1.27)) hide)
     )
@@
       (effects (font (size 1.27 1.27)) (justify left))
     )
-    (property "Footprint" "" (id 2) (at 226.06 53.34 0)
+    (property "Footprint" "solderwirepad_1_02_SMD:SolderWirePad_1x03_SMD_1x3mm" (id 2) (at 226.06 53.34 0)
       (effects (font (size 1.27 1.27)) hide)
     )
@@
     (property "Reference" "SW1" (id 0) (at 114.3 81.28 0))
     (property "Value" "Conn_01x02" (id 1) (at 114.3 83.82 0))
-    (property "Footprint" "" (id 2) (at 114.3 90.17 0)
+    (property "Footprint" "solderwirepad_1_02_SMD:SolderWirePad_1x02_SMD_5x5mm" (id 2) (at 114.3 90.17 0)
       (effects (font (size 1.27 1.27)) hide)
     )
@@
     (property "Reference" "SW4" (id 0) (at 170.18 93.98 0))
     (property "Value" "RotaryEncoder_Switch" (id 1) (at 170.18 96.52 0))
-    (property "Footprint" "" (id 2) (at 166.37 100.076 0)
+    (property "Footprint" "solderwirepad_1_02_SMD:SolderWirePad_1x05_SMD_1x3mm" (id 2) (at 166.37 100.076 0)
       (effects (font (size 1.27 1.27)) hide)
     )
@@
       (effects (font (size 1.27 1.27)) (justify left))
     )
-    (property "Footprint" "" (id 2) (at 161.29 72.39 0)
+    (property "Footprint" "solderwirepad_1_02_SMD:SolderWirePad_1x02_SMD_5x5mm" (id 2) (at 161.29 72.39 0)
       (effects (font (size 1.27 1.27)) hide)
     )
@@
     )
     (path "/c7504dc0-d4d5-4e17-89ac-603c04c71849"
-      (reference "B_RAW1") (unit 1) (value "Conn_01x02") (footprint "")
+      (reference "B_RAW1") (unit 1) (value "Conn_01x02") (footprint "solderwirepad_1_02_SMD:SolderWirePad_1x02_SMD_5x5mm")
     )
     (path "/31f0503a-7085-43d4-80f5-3276edea139e"
@@
     )
     (path "/1eb35198-95db-4c72-8594-cc447d0c72e9"
-      (reference "R1") (unit 1) (value "R") (footprint "")
+      (reference "R1") (unit 1) (value "R") (footprint "Resistor_THT:R_Axial_DIN0207_L6.3mm_D2.5mm_P7.62mm_Horizontal")
     )
     (path "/6b10fc84-89f0-4b5c-815b-3381303a3189"
-      (reference "SW1") (unit 1) (value "Conn_01x02") (footprint "")
+      (reference "SW1") (unit 1) (value "Conn_01x02") (footprint "solderwirepad_1_02_SMD:SolderWirePad_1x02_SMD_5x5mm")
     )
     (path "/2be7e24f-6eb6-4bab-af22-c76ca4f9f7fe"
-      (reference "SW2") (unit 1) (value "Conn_01x02") (footprint "")
+      (reference "SW2") (unit 1) (value "Conn_01x02") (footprint "solderwirepad_1_02_SMD:SolderWirePad_1x02_SMD_5x5mm")
     )
     (path "/2e30c3cf-1b1d-4f84-99c3-6155a5f74fd2"
-      (reference "SW3") (unit 1) (value "Conn_01x02") (footprint "")
+      (reference "SW3") (unit 1) (value "Conn_01x02") (footprint "solderwirepad_1_02_SMD:SolderWirePad_1x02_SMD_5x5mm")
     )
     (path "/b9262ad3-a2e5-4e5f-a098-530b7e584d34"
-      (reference "SW4") (unit 1) (value "RotaryEncoder_Switch") (footprint "")
+      (reference "SW4") (unit 1) (value "RotaryEncoder_Switch") (footprint "solderwirepad_1_02_SMD:SolderWirePad_1x05_SMD_1x3mm")
     )
     (path "/25910c11-2c64-427c-a074-9466462c9c63"
-      (reference "TP1") (unit 1) (value "Conn_01x04") (footprint "")
+      (reference "TP1") (unit 1) (value "Conn_01x04") (footprint "solderwirepad_1_02_SMD:SolderWirePad_1x04_SMD_1x3mm")
     )
     (path "/4bcbb00d-5a9e-4860-a7f1-1b9a042c53e8"
-      (reference "TPS1") (unit 1) (value "Conn_01x03") (footprint "")
+      (reference "TPS1") (unit 1) (value "Conn_01x03") (footprint "solderwirepad_1_02_SMD:SolderWirePad_1x03_SMD_1x3mm")
     )
     (path "/f1388b60-83a7-4b48-ade8-fa011085dd30"

Commit message: made some new footprtints soldering pad
Parts:
- A1: footprint solderwirepad_1_02_SMD:SolderWirePad_1x07_SMD_1x3mm -> solderwirepad_1_02_SMD:SolderWirePad_1x07_SMD_2x6mm
- B_RAW1, J1, PWR1, SW1, SW2, SW3: footprint solderwirepad_1_02_SMD:SolderWirePad_1x02_SMD_5x5mm -> solderwirepad_1_02_SMD:SolderWirePad_1x02_SMD_2x6mm
- M1: footprint solderwirepad_1_02_SMD:SolderWirePad_1x06_SMD_1x3mm -> solderwirepad_1_02_SMD:SolderWirePad_1x06_SMD_2x6mm
- OLED1: footprint solderwirepad_1_02_SMD:SolderWirePad_1x07_SMD_1x3mm -> solderwirepad_1_02_SMD:SolderWirePad_1x02_SMD_2x6mm
- SW4: footprint solderwirepad_1_02_SMD:SolderWirePad_1x05_SMD_1x3mm -> solderwirepad_1_02_SMD:SolderWirePad_1x05_SMD_2x6mm
- TP1: footprint solderwirepad_1_02_SMD:SolderWirePad_1x04_SMD_1x3mm -> solderwirepad_1_02_SMD:SolderWirePad_1x04_SMD_2x6mm
- TPS1: footprint solderwirepad_1_02_SMD:SolderWirePad_1x03_SMD_1x3mm -> solderwirepad_1_02_SMD:SolderWirePad_1x03_SMD_2x6mm
- U1: footprint ESP32-S3-DEVKITC-1U-N8R8:MODULE_ESP32-S3-DEVKITC-1U-N8R8 -> XIAO_ESP32C3:MODULE_ESP32_NODEMCU
Changed lines of the file:
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@@
+    )
+  )
+  (global_label "SW_RE" (shape input) (at 74.93 78.74 0) (fields_autoplaced)
+    (effects (font (size 1 1)) (justify left))
+    (property "Intersheet References" "${INTERSHEET_REFS}" (id 0) (at 81.5919 78.6775 0)
+      (effects (font (size 1 1)) (justify left) hide)
     )
   )
@@
       (effects (font (size 1.27 1.27)) (justify left))
     )
-    (property "Footprint" "solderwirepad_1_02_SMD:SolderWirePad_1x04_SMD_1x3mm" (id 2) (at 185.42 86.36 0)
+    (property "Footprint" "solderwirepad_1_02_SMD:SolderWirePad_1x04_SMD_2x6mm" (id 2) (at 185.42 86.36 0)
       (effects (font (size 1.27 1.27)) hide)
     )
@@
     (property "Reference" "SW2" (id 0) (at 135.89 81.28 0))
     (property "Value" "Conn_01x02" (id 1) (at 135.89 83.82 0))
-    (property "Footprint" "solderwirepad_1_02_SMD:SolderWirePad_1x02_SMD_5x5mm" (id 2) (at 135.89 90.17 0)
+    (property "Footprint" "solderwirepad_1_02_SMD:SolderWirePad_1x02_SMD_2x6mm" (id 2) (at 135.89 90.17 0)
       (effects (font (size 1.27 1.27)) hide)
     )
@@
     (property "Reference" "SW3" (id 0) (at 151.13 81.28 0))
     (property "Value" "Conn_01x02" (id 1) (at 151.13 83.82 0))
-    (property "Footprint" "solderwirepad_1_02_SMD:SolderWirePad_1x02_SMD_5x5mm" (id 2) (at 151.13 90.17 0)
+    (property "Footprint" "solderwirepad_1_02_SMD:SolderWirePad_1x02_SMD_2x6mm" (id 2) (at 151.13 90.17 0)
       (effects (font (size 1.27 1.27)) hide)
     )
@@
     (property "Reference" "J1" (id 0) (at 114.3 99.06 0))
     (property "Value" "Conn_01x02" (id 1) (at 114.3 101.6 0))
-    (property "Footprint" "solderwirepad_1_02_SMD:SolderWirePad_1x02_SMD_5x5mm" (id 2) (at 114.3 107.95 0)
+    (property "Footprint" "solderwirepad_1_02_SMD:SolderWirePad_1x02_SMD_2x6mm" (id 2) (at 114.3 107.95 0)
       (effects (font (size 1.27 1.27)) hide)
     )
@@
       (effects (font (size 1.27 1.27)) (justify left))
     )
-    (property "Footprint" "solderwirepad_1_02_SMD:SolderWirePad_1x03_SMD_1x3mm" (id 2) (at 226.06 53.34 0)
+    (property "Footprint" "solderwirepad_1_02_SMD:SolderWirePad_1x03_SMD_2x6mm" (id 2) (at 226.06 53.34 0)
       (effects (font (size 1.27 1.27)) hide)
     )
@@
       (effects (font (size 1.27 1.27)) (justify left))
     )
-    (property "Footprint" "solderwirepad_1_02_SMD:SolderWirePad_1x07_SMD_1x3mm" (id 2) (at 107.95 36.83 0)
+    (property "Footprint" "solderwirepad_1_02_SMD:SolderWirePad_1x02_SMD_2x6mm" (id 2) (at 107.95 36.83 0)
       (effects (font (size 1.27 1.27)) hide)
     )
@@
     (property "Reference" "PWR1" (id 0) (at 135.89 96.52 0))
     (property "Value" "Conn_01x02" (id 1) (at 135.89 99.06 0))
-    (property "Footprint" "solderwirepad_1_02_SMD:SolderWirePad_1x02_SMD_5x5mm" (id 2) (at 135.89 105.41 0)
+    (property "Footprint" "solderwirepad_1_02_SMD:SolderWirePad_1x02_SMD_2x6mm" (id 2) (at 135.89 105.41 0)
       (effects (font (size 1.27 1.27)) hide)
     )
@@
     (property "Reference" "SW1" (id 0) (at 114.3 81.28 0))
     (property "Value" "Conn_01x02" (id 1) (at 114.3 83.82 0))
-    (property "Footprint" "solderwirepad_1_02_SMD:SolderWirePad_1x02_SMD_5x5mm" (id 2) (at 114.3 90.17 0)
+    (property "Footprint" "solderwirepad_1_02_SMD:SolderWirePad_1x02_SMD_2x6mm" (id 2) (at 114.3 90.17 0)
       (effects (font (size 1.27 1.27)) hide)
     )
@@
     (property "Reference" "SW4" (id 0) (at 170.18 93.98 0))
     (property "Value" "RotaryEncoder_Switch" (id 1) (at 170.18 96.52 0))
-    (property "Footprint" "solderwirepad_1_02_SMD:SolderWirePad_1x05_SMD_1x3mm" (id 2) (at 166.37 100.076 0)
+    (property "Footprint" "solderwirepad_1_02_SMD:SolderWirePad_1x05_SMD_2x6mm" (id 2) (at 166.37 100.076 0)
       (effects (font (size 1.27 1.27)) hide)
     )
@@
       (effects (font (size 1.27 1.27)) (justify left))
     )
-    (property "Footprint" "solderwirepad_1_02_SMD:SolderWirePad_1x06_SMD_1x3mm" (id 2) (at 104.14 63.5 0)
+    (property "Footprint" "solderwirepad_1_02_SMD:SolderWirePad_1x06_SMD_2x6mm" (id 2) (at 104.14 63.5 0)
       (effects (font (size 1.27 1.27)) hide)
     )
@@
       (effects (font (size 1.27 1.27)) (justify left))
     )
-    (property "Footprint" "solderwirepad_1_02_SMD:SolderWirePad_1x02_SMD_5x5mm" (id 2) (at 161.29 72.39 0)
+    (property "Footprint" "solderwirepad_1_02_SMD:SolderWirePad_1x02_SMD_2x6mm" (id 2) (at 161.29 72.39 0)
       (effects (font (size 1.27 1.27)) hide)
     )
@@
     (property "Reference" "U1" (id 0) (at 52.0738 20.32 0))
     (property "Value" "ESP32-38_pins" (id 1) (at 52.0738 22.86 0))
-    (property "Footprint" "ESP32-S3-DEVKITC-1U-N8R8:MODULE_ESP32-S3-DEVKITC-1U-N8R8" (id 2) (at -22.86 22.86 0)
+    (property "Footprint" "XIAO_ESP32C3:MODULE_ESP32_NODEMCU" (id 2) (at -22.86 22.86 0)
       (effects (font (size 1.27 1.27)) (justify bottom) hide)
     )
@@
       (effects (font (size 1.27 1.27)) (justify left))
     )
-    (property "Footprint" "solderwirepad_1_02_SMD:SolderWirePad_1x07_SMD_1x3mm" (id 2) (at 156.21 36.83 0)
+    (property "Footprint" "solderwirepad_1_02_SMD:SolderWirePad_1x07_SMD_2x6mm" (id 2) (at 156.21 36.83 0)
       (effects (font (size 1.27 1.27)) hide)
     )
@@
   (symbol_instances
     (path "/fa96dc13-12ef-485e-89f3-d951ded670b6"
-      (reference "A1") (unit 1) (value "Conn_01x07") (footprint "solderwirepad_1_02_SMD:SolderWirePad_1x07_SMD_1x3mm")
+      (reference "A1") (unit 1) (value "Conn_01x07") (footprint "solderwirepad_1_02_SMD:SolderWirePad_1x07_SMD_2x6mm")
     )
     (path "/c7504dc0-d4d5-4e17-89ac-603c04c71849"
-      (reference "B_RAW1") (unit 1) (value "Conn_01x02") (footprint "solderwirepad_1_02_SMD:SolderWirePad_1x02_SMD_5x5mm")
+      (reference "B_RAW1") (unit 1) (value "Conn_01x02") (footprint "solderwirepad_1_02_SMD:SolderWirePad_1x02_SMD_2x6mm")
     )
     (path "/31f0503a-7085-43d4-80f5-3276edea139e"
-      (reference "J1") (unit 1) (value "Conn_01x02") (footprint "solderwirepad_1_02_SMD:SolderWirePad_1x02_SMD_5x5mm")
+      (reference "J1") (unit 1) (value "Conn_01x02") (footprint "solderwirepad_1_02_SMD:SolderWirePad_1x02_SMD_2x6mm")
     )
     (path "/baaea415-07fe-418e-aedc-efe7b02c604a"
-      (reference "M1") (unit 1) (value "Conn_01x06") (footprint "solderwirepad_1_02_SMD:SolderWirePad_1x06_SMD_1x3mm")
+      (reference "M1") (unit 1) (value "Conn_01x06") (footprint "solderwirepad_1_02_SMD:SolderWirePad_1x06_SMD_2x6mm")
     )
     (path "/5880f81e-0533-41b0-b0fb-73380c5496c7"
-      (reference "OLED1") (unit 1) (value "Conn_01x07") (footprint "solderwirepad_1_02_SMD:SolderWirePad_1x07_SMD_1x3mm")
+      (reference "OLED1") (unit 1) (value "Conn_01x07") (footprint "solderwirepad_1_02_SMD:SolderWirePad_1x02_SMD_2x6mm")
     )
     (path "/5977c44d-5ca0-4b6f-9afe-957b1d414631"
-      (reference "PWR1") (unit 1) (value "Conn_01x02") (footprint "solderwirepad_1_02_SMD:SolderWirePad_1x02_SMD_5x5mm")
+      (reference "PWR1") (unit 1) (value "Conn_01x02") (footprint "solderwirepad_1_02_SMD:SolderWirePad_1x02_SMD_2x6mm")
     )
     (path "/1eb35198-95db-4c72-8594-cc447d0c72e9"
@@
     )
     (path "/6b10fc84-89f0-4b5c-815b-3381303a3189"
-      (reference "SW1") (unit 1) (value "Conn_01x02") (footprint "solderwirepad_1_02_SMD:SolderWirePad_1x02_SMD_5x5mm")
+      (reference "SW1") (unit 1) (value "Conn_01x02") (footprint "solderwirepad_1_02_SMD:SolderWirePad_1x02_SMD_2x6mm")
     )
     (path "/2be7e24f-6eb6-4bab-af22-c76ca4f9f7fe"
-      (reference "SW2") (unit 1) (value "Conn_01x02") (footprint "solderwirepad_1_02_SMD:SolderWirePad_1x02_SMD_5x5mm")
+      (reference "SW2") (unit 1) (value "Conn_01x02") (footprint "solderwirepad_1_02_SMD:SolderWirePad_1x02_SMD_2x6mm")
     )
     (path "/2e30c3cf-1b1d-4f84-99c3-6155a5f74fd2"
-      (reference "SW3") (unit 1) (value "Conn_01x02") (footprint "solderwirepad_1_02_SMD:SolderWirePad_1x02_SMD_5x5mm")
+      (reference "SW3") (unit 1) (value "Conn_01x02") (footprint "solderwirepad_1_02_SMD:SolderWirePad_1x02_SMD_2x6mm")
     )
     (path "/b9262ad3-a2e5-4e5f-a098-530b7e584d34"
-      (reference "SW4") (unit 1) (value "RotaryEncoder_Switch") (footprint "solderwirepad_1_02_SMD:SolderWirePad_1x05_SMD_1x3mm")
+      (reference "SW4") (unit 1) (value "RotaryEncoder_Switch") (footprint "solderwirepad_1_02_SMD:SolderWirePad_1x05_SMD_2x6mm")
     )
     (path "/25910c11-2c64-427c-a074-9466462c9c63"
-      (reference "TP1") (unit 1) (value "Conn_01x04") (footprint "solderwirepad_1_02_SMD:SolderWirePad_1x04_SMD_1x3mm")
+      (reference "TP1") (unit 1) (value "Conn_01x04") (footprint "solderwirepad_1_02_SMD:SolderWirePad_1x04_SMD_2x6mm")
     )
     (path "/4bcbb00d-5a9e-4860-a7f1-1b9a042c53e8"
-      (reference "TPS1") (unit 1) (value "Conn_01x03") (footprint "solderwirepad_1_02_SMD:SolderWirePad_1x03_SMD_1x3mm")
+      (reference "TPS1") (unit 1) (value "Conn_01x03") (footprint "solderwirepad_1_02_SMD:SolderWirePad_1x03_SMD_2x6mm")
     )
     (path "/f1388b60-83a7-4b48-ade8-fa011085dd30"
-      (reference "U1") (unit 1) (value "ESP32-38_pins") (footprint "ESP32-S3-DEVKITC-1U-N8R8:MODULE_ESP32-S3-DEVKITC-1U-N8R8")
-    )
-  )
+      (reference "U1") (unit 1) (value "ESP32-38_pins") (footprint "XIAO_ESP32C3:MODULE_ESP32_NODEMCU")
+    )
+  )

Commit message: routing half way
Parts:
- A1: value Conn_01x07 -> A1
- B_RAW1: value Conn_01x02 -> B_RAW
- J1: value Conn_01x02 -> J1
- M1: value Conn_01x06 -> M1
- OLED1: value Conn_01x07 -> OLED; footprint solderwirepad_1_02_SMD:SolderWirePad_1x02_SMD_2x6mm -> solderwirepad_1_02_SMD:SolderWirePad_1x07_SMD_2x6mm
- PWR1: value Conn_01x02 -> PWR
- SW1: value Conn_01x02 -> SW1
- SW2: value Conn_01x02 -> SW2
- SW3: value Conn_01x02 -> SW3
- TP1: value Conn_01x04 -> TP1
- TPS1: value Conn_01x03 -> TPS1
Connections:
- net L/R is gone; now on net GND: M1.6 (Pin_6), U1.J2_7 (GND)
- net CS: now also U1.J2_12 (GPIO16); no longer U1.J1_12 (GPIO16)
- net GND: now also SW4.3 (C), SW4.5 (S2); no longer SW4.C, SW4.S2
- net RE_A: now also SW4.1 (A); no longer SW4.A
- net RE_B: now also SW4.2 (B); no longer SW4.B
- net SW_RE: now also SW4.4 (S1); no longer SW4.S1
- net SW3: no longer names the net of SW3.2 (Pin_2), U1.J1_12 (GPIO14)
Other:
- moved on the sheet: SW3
