File: phone/phone.kicad_pcb (KiCad board)
At the start: 2 copper layers, 14 parts, among them J1 Conn_01x02, M1 Conn_01x06, SW1 Conn_01x02, SW2 Conn_01x02, SW3 Conn_01x02, SW4 RotaryEncoder_Switch, U1 ESP32-38_pins

Commit message: routing half way
Parts:
- A1: value Conn_01x07 -> A1
- B_RAW1: value Conn_01x02 -> B_RAW
- J1: value Conn_01x02 -> J1
- M1: value Conn_01x06 -> M1; moved to B.Cu
- OLED1: value Conn_01x07 -> OLED; footprint solderwirepad_1_02_SMD:SolderWirePad_1x02_SMD_2x6mm -> solderwirepad_1_02_SMD:SolderWirePad_1x07_SMD_2x6mm
- PWR1: value Conn_01x02 -> PWR
- SW1: value Conn_01x02 -> SW1
- SW2: value Conn_01x02 -> SW2
- SW3: value Conn_01x02 -> SW3
- TP1: value Conn_01x04 -> TP1; moved to B.Cu
- TPS1: value Conn_01x03 -> TPS1; moved to B.Cu
- moved PWR1 133.1 mm to (37.4, 82.2)
- moved TPS1 123.7 mm to (42.2, 83.4), turned to 180 degrees
- moved M1 115.8 mm to (47.5, 48.2), turned to 90 degrees
- moved TP1 106.9 mm to (42.7, 75.6), turned to 180 degrees
- moved B_RAW1 105.2 mm to (43.9, 61.7), turned to 90 degrees
- moved R1 101.9 mm to (52.2, 32.3), turned to 180 degrees
- moved SW1 82.4 mm to (36.7, 70.1), turned to 180 degrees
- moved SW3 76.1 mm to (48.3, 82.6)
- moved J1 75.4 mm to (41.9, 40.3), turned to -90 degrees
- moved OLED1 70.3 mm to (49.9, 54.5), turned to -90 degrees
- moved SW2 66.0 mm to (41.6, 51.0), turned to -90 degrees
- moved SW4 55.2 mm to (35.5, 43.4), turned to -90 degrees
Connections:
- M1 pad 6: L/R -> GND
- SW3 pad 2: SW3 -> Net-(SW3-Pad2)
- SW4 pad 1: (no net) -> RE_A
- SW4 pad 2: (no net) -> RE_B
- SW4 pad 3: (no net) -> GND
- SW4 pad 4: (no net) -> SW_RE
- SW4 pad 5: (no net) -> GND
- U1 pad J1_12: CS -> Net-(SW3-Pad2)
- U1 pad J2_12: (no net) -> CS
- U1 pad J2_13: (no net) -> unconnected-(U1-PadJ2_13)
- U1 pad J2_7: L/R -> GND
Routing:
- net RE_B: track 0.00 -> 140.2 mm
- net GND: track 0.00 -> 92.0 mm, vias 0 -> 2
- net RE_A: track 0.00 -> 75.3 mm
- net LED: track 0.00 -> 50.1 mm
- net 3V3: track 0.00 -> 39.1 mm, vias 0 -> 1
- net RST: track 0.00 -> 32.2 mm
- net DC: track 0.00 -> 21.6 mm
- net DIN: track 0.00 -> 15.7 mm
- net CS: track 0.00 -> 6.27 mm
- net CLK: track 0.00 -> 5.36 mm
- net VIN: track 0.00 -> 4.09 mm
- net SW1: track 0.00 -> 3.52 mm

Commit message: routing done
Parts:
- moved SW1 0.33 mm to (37.1, 70.0)
- moved SW4 0.28 mm to (35.5, 43.1)
Routing:
- net 3V3: track 39.1 -> 109.1 mm, vias 1 -> 3
- net WS: track 0.00 -> 56.0 mm
- net Net-(SW3-Pad2): track 0.00 -> 54.6 mm
- net GND: track 92.0 -> 136.0 mm, vias 2 -> 5
- net BAT_BOOST: track 0.00 -> 29.2 mm
- net SD: track 0.00 -> 22.4 mm
- net SCK: track 0.00 -> 20.9 mm
- net Net-(J1-Pad2): track 0.00 -> 18.8 mm
- net SW2: track 0.00 -> 17.1 mm
- net BAT_RAW: track 0.00 -> 11.4 mm, vias 0 -> 1
- net A1_DIN: track 0.00 -> 9.44 mm
- net VIN: track 4.09 -> 7.85 mm, vias 0 -> 1
- net (no net): track 0.00 -> 0.96 mm
Other:
- board outline added: 39.3 x 65 mm
